File: hardware/main_controller/portde.sch (KiCad schematic (older format))
At the start: 2 parts

Commit message: Assigned names
Parts:
- gave numbers to parts that had none: 1
Changed lines of the file:
@@
 $EndDescr
 $Comp
-L stm32:STM32F407V(E-G)Tx_u U?
+L stm32:STM32F407V(E-G)Tx_u U1
 U 4 1 5FDB9E32
 P 2400 1800
-F 0 "U?" H 2407 2957 50  0000 C CNN
+F 0 "U1" H 2407 2957 50  0000 C CNN
 F 1 "STM32F407V(E-G)Tx_u" H 2407 2866 50  0000 C CNN
 F 2 "LQFP100" H 2407 2775 50  0000 C CIN
@@
 CAN_TX
 $Comp
-L stm32:STM32F407V(E-G)Tx_u U?
+L stm32:STM32F407V(E-G)Tx_u U1
 U 5 1 5FE25B58
 P 2400 3900
-F 0 "U?" H 2407 5057 50  0000 C CNN
+F 0 "U1" H 2407 5057 50  0000 C CNN
 F 1 "STM32F407V(E-G)Tx_u" H 2407 4966 50  0000 C CNN
 F 2 "LQFP100" H 2407 4875 50  0000 C CIN

Commit message: assigned footprints
Parts:
- U1: footprint LQFP100 -> Package_QFP:LQFP-100_14x14mm_P0.5mm
Changed lines of the file:
@@
 F 0 "U1" H 2407 2957 50  0000 C CNN
 F 1 "STM32F407V(E-G)Tx_u" H 2407 2866 50  0000 C CNN
-F 2 "LQFP100" H 2407 2775 50  0000 C CIN
+F 2 "Package_QFP:LQFP-100_14x14mm_P0.5mm" H 2407 2775 50  0000 C CIN
 F 3 "" H 2400 1800 50  0000 C CNN
 	4    2400 1800
@@
 F 0 "U1" H 2407 5057 50  0000 C CNN
 F 1 "STM32F407V(E-G)Tx_u" H 2407 4966 50  0000 C CNN
-F 2 "LQFP100" H 2407 4875 50  0000 C CIN
+F 2 "Package_QFP:LQFP-100_14x14mm_P0.5mm" H 2407 4875 50  0000 C CIN
 F 3 "" H 2400 3900 50  0000 C CNN
 	5    2400 3900
