File: hardware/main_controller/connectivity.sch (KiCad schematic (older format))
At the start: 37 parts, among them J1 USB_B_Mini, J10 JTAG_Connector, J11 RJ45, J12 RJ45, J2 USB_C_Receptacle_USB2.0, J3 GPIO_1, J4 GPIO_2, J5 GPIO_PWR_1, J6 I2C, J7 GPIO_PWR_2, J8 SPI, J9 SPI_PWR, U2 MCP2551-I-SN, U4 USBLC6-2SC6

Commit message: pcb
Parts:
- JP1: footprint Connector_PinSocket_2.54mm:PinSocket_1x03_P2.54mm_Vertical -> Connector_PinHeader_2.54mm:PinHeader_1x03_P2.54mm_Vertical
- JP2, JP3, JP4: footprint Connector_PinSocket_2.54mm:PinSocket_1x02_P2.54mm_Vertical -> Connector_PinHeader_2.54mm:PinHeader_1x02_P2.54mm_Vertical
Connections:
- net DM: now also J1.2 (D-)
- net DP: now also J1.3 (D+)
- net USB_DM: no longer J1.2 (D-)
- net USB_DP: no longer J1.3 (D+)
Changed lines of the file:
@@
 	900  3850 900  4000
 Connection ~ 900  3850
-Text GLabel 1450 3450 2    50   Input ~ 0
-USB_DP
-Text GLabel 1450 3550 2    50   Input ~ 0
-USB_DM
 $Comp
 L Device:R R5
@@
 F 0 "JP3" V 8154 4398 50  0000 L CNN
 F 1 "JMP_CAN_TERM" V 8245 4398 50  0000 L CNN
-F 2 "Connector_PinSocket_2.54mm:PinSocket_1x02_P2.54mm_Vertical" H 8200 4350 50  0001 C CNN
+F 2 "Connector_PinHeader_2.54mm:PinHeader_1x02_P2.54mm_Vertical" H 8200 4350 50  0001 C CNN
 F 3 "~" H 8200 4350 50  0001 C CNN
 	1    8200 4350
@@
 F 0 "JP2" H 7600 3885 50  0000 C CNN
 F 1 "JMP_CAN_PWR" H 7600 3794 50  0000 C CNN
-F 2 "Connector_PinSocket_2.54mm:PinSocket_1x02_P2.54mm_Vertical" H 7600 3700 50  0001 C CNN
+F 2 "Connector_PinHeader_2.54mm:PinHeader_1x02_P2.54mm_Vertical" H 7600 3700 50  0001 C CNN
 F 3 "~" H 7600 3700 50  0001 C CNN
 	1    7600 3700
@@
 F 0 "JP4" V 4804 1498 50  0000 L CNN
 F 1 "JMP_USB_PU" V 4895 1498 50  0000 L CNN
-F 2 "Connector_PinSocket_2.54mm:PinSocket_1x02_P2.54mm_Vertical" H 4850 1450 50  0001 C CNN
+F 2 "Connector_PinHeader_2.54mm:PinHeader_1x02_P2.54mm_Vertical" H 4850 1450 50  0001 C CNN
 F 3 "~" H 4850 1450 50  0001 C CNN
 	1    4850 1450
@@
 F 0 "JP1" V 3904 2767 50  0000 L CNN
 F 1 "JMP_USB_PWR" V 3995 2767 50  0000 L CNN
-F 2 "Connector_PinSocket_2.54mm:PinSocket_1x03_P2.54mm_Vertical" H 3950 2700 50  0001 C CNN
+F 2 "Connector_PinHeader_2.54mm:PinHeader_1x03_P2.54mm_Vertical" H 3950 2700 50  0001 C CNN
 F 3 "~" H 3950 2700 50  0001 C CNN
 	1    3950 2700
@@
 Wire Wire Line
 	3450 2400 3550 2400
+Text GLabel 1450 3450 2    50   Input ~ 0
+DP
+Text GLabel 1450 3550 2    50   Input ~ 0
+DM
 $EndSCHEMATC
